File: MainModule/PCB/MainModule/mainModule.sch (EAGLE design)
At the start: 20 parts, among them U1 LM5007MM, U2 LM3940IMP-3.3, X2 MINI-USB-32005-201

Commit message: Replacing schematic for switching supply in to new document PowerSupplyModule/PCB/powerSupplyModule.sch
Parts:
- removed C1: 1uF, 100V, resistor:CPOL-EU153CLV-0405
- removed C2: 15uF, 25V, resistor:CPOL-EUC
- removed C3: 100nF, 50V, resistor:CPOL-EUSMCA
- removed C4: 10nF, 50V, resistor:CPOL-EUR/2012-12W
- removed C5: 100nF, 100V, resistor:CPOL-EUSMCA
- removed D1: 1N4148DO35-7, diode:1N4148DO35-7
- removed L1: 100uH, inductor-neosid:SM-Z15
- removed R1: 200K, rcl:R-EU_R2010
- removed R2: 100K, rcl:R-EU_R2010
- removed R3, R4: 1K, rcl:R-EU_R2010
- removed R5: 1ohm, rcl:R-EU_R2010
- removed U1: LM5007MM, LM5007:LM5007MM
- removed VIN: 12-75V, con-molex:5566-2
Connections:
- removed net N$1: R2.2, U1.RCL
- removed net N$3: R1.1, U1.RON
- removed net N$5: C4.+, U1.BST
- removed net N$6: C4.-, D1.C, L1.1, U1.SW
- removed net N$7: C3.+, U1.VCC
- removed net N$8: R3.1, R4.2, U1.FEEDBACK
- removed net N$9: C2.+, R5.1
- removed net VIN(12-75V): C1.+, C5.+, R1.2, U1.VIN, VIN-2.S
- net GND: no longer C1.-, C2.-, C3.-, C5.-, D1.A, R2.1, R4.1, U1.RTN, VIN-1.S
- net U(5V): no longer L1.2, R3.2, R5.2
