File: ControlExpansionModule/PCB/ControlExpansionModule/CEM-8bit-PCA9557.sch (EAGLE design)
At the start: 0 parts

Commit message: Wired schematic for port expander, based on PCA9557
Parts:
- added R1, R2: 1.8K, resistor:R-EU_MELF0204R
- added R3, R4: 2K, resistor:R-EU_MELF0204R
- added U1: PCA9557D, PCA9557:PCA9557D
- added X1: power/communicatino-connector, con-molex:43160-1104
Connections:
- new net GND: U1.VSS, X1-1.S@1
- new net N$3: R3.1, U1.!RESET
- new net SCL: R1.1, U1.SCL, X1-3.S@1
- new net SDA: R2.1, U1.SDA, X1-2.S@1
- new net VCC: R1.2, R2.2, R3.2, R4.2, U1.VDD, X1-4.S@1
Changed lines of the file:
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@@
 <parts>
 <part name="FRAME1" library="frames" deviceset="A4L-LOC" device=""/>
+<part name="U1" library="PCA9557" deviceset="PCA9557D" device=""/>
+<part name="R1" library="resistor" deviceset="R-EU_" device="MELF0204R" value="1.8K"/>
+<part name="R2" library="resistor" deviceset="R-EU_" device="MELF0204R" value="1.8K"/>
+<part name="R3" library="resistor" deviceset="R-EU_" device="MELF0204R" value="2K"/>
+<part name="R4" library="resistor" deviceset="R-EU_" device="MELF0204R" value="2K"/>
+<part name="X1" library="con-molex" deviceset="43160-*04" device="" technology="11" value="power/communicatino-connector"/>
+<part name="GND1" library="supply1" deviceset="GND" device=""/>
+<part name="P+1" library="supply1" deviceset="VCC" device=""/>
+<part name="P+2" library="supply1" deviceset="VCC" device=""/>
+<part name="GND2" library="supply1" deviceset="GND" device=""/>
 </parts>
 <sheets>
@@
 <instances>
 <instance part="FRAME1" gate="G$1" x="0" y="0"/>
+<instance part="U1" gate="A" x="162.56" y="88.9"/>
+<instance part="R1" gate="G$1" x="88.9" y="101.6" rot="R90"/>
+<instance part="R2" gate="G$1" x="101.6" y="101.6" rot="R90"/>
+<instance part="R3" gate="G$1" x="114.3" y="101.6" rot="R90"/>
+<instance part="R4" gate="G$1" x="127" y="101.6" rot="R90"/>
+<instance part="X1" gate="-1" x="60.96" y="88.9" rot="R180"/>
+<instance part="X1" gate="-2" x="60.96" y="91.44" rot="R180"/>
+<instance part="X1" gate="-3" x="60.96" y="93.98" rot="R180"/>
+<instance part="X1" gate="-4" x="60.96" y="96.52" rot="R180"/>
+<instance part="GND1" gate="1" x="68.58" y="83.82"/>
+<instance part="P+1" gate="VCC" x="68.58" y="104.14"/>
+<instance part="P+2" gate="VCC" x="144.78" y="121.92"/>
+<instance part="GND2" gate="1" x="142.24" y="63.5"/>
 </instances>
 <busses>
 </busses>
 <nets>
+<net name="VCC" class="0">
+<segment>
+<pinref part="P+1" gate="VCC" pin="VCC"/>
+<pinref part="X1" gate="-4" pin="S@1"/>
+<wire x1="68.58" y1="101.6" x2="68.58" y2="96.52" width="0.1524" layer="91"/>
+<wire x1="68.58" y1="96.52" x2="66.04" y2="96.52" width="0.1524" layer="91"/>
+<wire x1="68.58" y1="104.14" x2="68.58" y2="101.6" width="0.1524" layer="91"/>
+</segment>
+<segment>
+<pinref part="P+2" gate="VCC" pin="VCC"/>
+<wire x1="144.78" y1="119.38" x2="144.78" y2="106.68" width="0.1524" layer="91"/>
+<pinref part="R1" gate="G$1" pin="2"/>
+<pinref part="U1" gate="A" pin="VDD"/>
+<wire x1="88.9" y1="106.68" x2="101.6" y2="106.68" width="0.1524" layer="91"/>
+<wire x1="101.6" y1="106.68" x2="114.3" y2="106.68" width="0.1524" layer="91"/>
+<wire x1="114.3" y1="106.68" x2="127" y2="106.68" width="0.1524" layer="91"/>
+<wire x1="127" y1="106.68" x2="144.78" y2="106.68" width="0.1524" layer="91"/>
+<wire x1="144.78" y1="106.68" x2="144.78" y2="99.06" width="0.1524" layer="91"/>
+<pinref part="R2" gate="G$1" pin="2"/>
+<junction x="101.6" y="106.68"/>
+<pinref part="R3" gate="G$1" pin="2"/>
+<junction x="114.3" y="106.68"/>
+<pinref part="R4" gate="G$1" pin="2"/>
+<junction x="127" y="106.68"/>
+<junction x="144.78" y="106.68"/>
+</segment>
+</net>
+<net name="GND" class="0">
+<segment>
+<pinref part="X1" gate="-1" pin="S@1"/>
+<pinref part="GND1" gate="1" pin="GND"/>
+<wire x1="66.04" y1="88.9" x2="68.58" y2="88.9" width="0.1524" layer="91"/>
+<wire x1="68.58" y1="88.9" x2="68.58" y2="86.36" width="0.1524" layer="91"/>
+</segment>
+<segment>
+<pinref part="U1" gate="A" pin="VSS"/>
+<pinref part="GND2" gate="1" pin="GND"/>
+<wire x1="144.78" y1="71.12" x2="142.24" y2="71.12" width="0.1524" layer="91"/>
+<wire x1="142.24" y1="71.12" x2="142.24" y2="66.04" width="0.1524" layer="91"/>
+</segment>
+</net>
+<net name="SCL" class="0">
+<segment>
+<pinref part="X1" gate="-3" pin="S@1"/>
+<wire x1="66.04" y1="93.98" x2="73.66" y2="93.98" width="0.1524" layer="91"/>
+<label x="71.12" y="93.98" size="1.778" layer="95"/>
+</segment>
+<segment>
+<pinref part="U1" gate="A" pin="SCL"/>
+<wire x1="144.78" y1="93.98" x2="88.9" y2="93.98" width="0.1524" layer="91"/>
+<pinref part="R1" gate="G$1" pin="1"/>
+<wire x1="88.9" y1="93.98" x2="73.66" y2="93.98" width="0.1524" layer="91"/>
+<wire x1="88.9" y1="96.52" x2="88.9" y2="93.98" width="0.1524" layer="91"/>
+<junction x="88.9" y="93.98"/>
+</segment>
+</net>
+<net name="SDA" class="0">
+<segment>
+<pinref part="X1" gate="-2" pin="S@1"/>
+<wire x1="66.04" y1="91.44" x2="73.66" y2="91.44" width="0.1524" layer="91"/>
+<label x="71.12" y="91.44" size="1.778" layer="95"/>
+</segment>
+<segment>
+<pinref part="U1" gate="A" pin="SDA"/>
+<wire x1="144.78" y1="91.44" x2="101.6" y2="91.44" width="0.1524" layer="91"/>
+<pinref part="R2" gate="G$1" pin="1"/>
+<wire x1="101.6" y1="91.44" x2="73.66" y2="91.44" width="0.1524" layer="91"/>
+<wire x1="101.6" y1="96.52" x2="101.6" y2="91.44" width="0.1524" layer="91"/>
+<junction x="101.6" y="91.44"/>
+</segment>
+</net>
+<net name="N$3" class="0">
+<segment>
+<pinref part="U1" gate="A" pin="!RESET"/>
+<pinref part="R3" gate="G$1" pin="1"/>
+<wire x1="144.78" y1="86.36" x2="114.3" y2="86.36" width="0.1524" layer="91"/>
+<wire x1="114.3" y1="86.36" x2="114.3" y2="96.52" width="0.1524" layer="91"/>
+</segment>
+</net>
 </nets>
 </sheet>
