File: ControlExpansionModule/PCB/ControlExpansionModule/CEM-16bit-PCF8575.sch (EAGLE design)
At the start: 0 parts

Commit message: Wiring component of the circuit of Port Expansion Module, based on PCF8575
Parts:
- added C1, C2: 50pF, rcl:C-EUC1206K
- added R1, R2: 1K, resistor:R-EU_M1406
- added R3: 2K, resistor:R-EU_M1406
- added U1: PCF8575PWE4, PCF8575:PCF8575PWE4
- added X1: 43160-1204, con-molex:43160-1204
Connections:
- new net GND: C1.2, C2.2, U1.A1, U1.A2, U1.GND, X1-1.S@1
- new net N$3: R3.1, U1.A0
- new net SCL: C1.1, R1.1, U1.SCL, X1-3.S@1
- new net SDA: C2.1, R2.1, U1.SDA, X1-2.S@1
- new net VCC: R1.2, R2.2, R3.2, U1.VCC, X1-4.S@1
Changed lines of the file:
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@@
 <parts>
 <part name="FRAME1" library="frames" deviceset="A4L-LOC" device=""/>
+<part name="U1" library="PCF8575" deviceset="PCF8575PWE4" device=""/>
+<part name="GND1" library="supply1" deviceset="GND" device=""/>
+<part name="GND2" library="supply1" deviceset="GND" device=""/>
+<part name="P+1" library="supply1" deviceset="VCC" device=""/>
+<part name="P+2" library="supply1" deviceset="VCC" device=""/>
+<part name="X1" library="con-molex" deviceset="43160-*04" device="" technology="12"/>
+<part name="C1" library="rcl" deviceset="C-EU" device="C1206K" value="50pF"/>
+<part name="R1" library="resistor" deviceset="R-EU_" device="M1406" value="1K"/>
+<part name="R2" library="resistor" deviceset="R-EU_" device="M1406" value="1K"/>
+<part name="C2" library="rcl" deviceset="C-EU" device="C1206K" value="50pF"/>
+<part name="R3" library="resistor" deviceset="R-EU_" device="M1406" value="2K"/>
+<part name="GND3" library="supply1" deviceset="GND" device=""/>
 </parts>
 <sheets>
@@
 <instances>
 <instance part="FRAME1" gate="G$1" x="0" y="0"/>
+<instance part="U1" gate="A" x="157.48" y="88.9"/>
+<instance part="GND1" gate="1" x="134.62" y="58.42"/>
+<instance part="GND2" gate="1" x="78.74" y="91.44"/>
+<instance part="P+1" gate="VCC" x="78.74" y="111.76"/>
+<instance part="P+2" gate="VCC" x="137.16" y="121.92"/>
+<instance part="X1" gate="-1" x="71.12" y="96.52" rot="R180"/>
+<instance part="X1" gate="-2" x="71.12" y="99.06" rot="R180"/>
+<instance part="X1" gate="-3" x="71.12" y="101.6" rot="R180"/>
+<instance part="X1" gate="-4" x="71.12" y="104.14" rot="R180"/>
+<instance part="C1" gate="G$1" x="96.52" y="88.9"/>
+<instance part="R1" gate="G$1" x="96.52" y="106.68" rot="R90"/>
+<instance part="R2" gate="G$1" x="109.22" y="106.68" rot="R90"/>
+<instance part="C2" gate="G$1" x="109.22" y="88.9"/>
+<instance part="R3" gate="G$1" x="129.54" y="106.68" rot="R90"/>
+<instance part="GND3" gate="1" x="101.6" y="76.2"/>
 </instances>
 <busses>
 </busses>
 <nets>
+<net name="VCC" class="0">
+<segment>
+<pinref part="P+1" gate="VCC" pin="VCC"/>
+<pinref part="X1" gate="-4" pin="S@1"/>
+<wire x1="78.74" y1="109.22" x2="78.74" y2="104.14" width="0.1524" layer="91"/>
+<wire x1="78.74" y1="104.14" x2="76.2" y2="104.14" width="0.1524" layer="91"/>
+</segment>
+<segment>
+<pinref part="P+2" gate="VCC" pin="VCC"/>
+<pinref part="U1" gate="A" pin="VCC"/>
+<wire x1="137.16" y1="119.38" x2="137.16" y2="111.76" width="0.1524" layer="91"/>
+<wire x1="137.16" y1="111.76" x2="137.16" y2="106.68" width="0.1524" layer="91"/>
+<wire x1="137.16" y1="106.68" x2="139.7" y2="106.68" width="0.1524" layer="91"/>
+<pinref part="R1" gate="G$1" pin="2"/>
+<wire x1="96.52" y1="111.76" x2="109.22" y2="111.76" width="0.1524" layer="91"/>
+<pinref part="R2" gate="G$1" pin="2"/>
+<junction x="109.22" y="111.76"/>
+<wire x1="109.22" y1="111.76" x2="129.54" y2="111.76" width="0.1524" layer="91"/>
+<junction x="137.16" y="111.76"/>
+<pinref part="R3" gate="G$1" pin="2"/>
+<wire x1="129.54" y1="111.76" x2="137.16" y2="111.76" width="0.1524" layer="91"/>
+<junction x="129.54" y="111.76"/>
+</segment>
+</net>
+<net name="GND" class="0">
+<segment>
+<pinref part="X1" gate="-1" pin="S@1"/>
+<pinref part="GND2" gate="1" pin="GND"/>
+<wire x1="76.2" y1="96.52" x2="78.74" y2="96.52" width="0.1524" layer="91"/>
+<wire x1="78.74" y1="96.52" x2="78.74" y2="93.98" width="0.1524" layer="91"/>
+</segment>
+<segment>
+<pinref part="U1" gate="A" pin="GND"/>
+<pinref part="GND1" gate="1" pin="GND"/>
+<wire x1="139.7" y1="63.5" x2="134.62" y2="63.5" width="0.1524" layer="91"/>
+<wire x1="134.62" y1="63.5" x2="134.62" y2="60.96" width="0.1524" layer="91"/>
+<pinref part="U1" gate="A" pin="A1"/>
+<wire x1="139.7" y1="93.98" x2="134.62" y2="93.98" width="0.1524" layer="91"/>
+<wire x1="134.62" y1="93.98" x2="134.62" y2="91.44" width="0.1524" layer="91"/>
+<pinref part="U1" gate="A" pin="A2"/>
+<wire x1="134.62" y1="91.44" x2="134.62" y2="63.5" width="0.1524" layer="91"/>
+<wire x1="139.7" y1="91.44" x2="134.62" y2="91.44" width="0.1524" layer="91"/>
+<junction x="134.62" y="63.5"/>
+<junction x="134.62" y="91.44"/>
+</segment>
+<segment>
+<pinref part="C1" gate="G$1" pin="2"/>
+<wire x1="96.52" y1="83.82" x2="96.52" y2="81.28" width="0.1524" layer="91"/>
+<wire x1="96.52" y1="81.28" x2="101.6" y2="81.28" width="0.1524" layer="91"/>
+<pinref part="C2" gate="G$1" pin="2"/>
+<wire x1="101.6" y1="81.28" x2="109.22" y2="81.28" width="0.1524" layer="91"/>
+<wire x1="109.22" y1="81.28" x2="109.22" y2="83.82" width="0.1524" layer="91"/>
+<pinref part="GND3" gate="1" pin="GND"/>
+<wire x1="101.6" y1="78.74" x2="101.6" y2="81.28" width="0.1524" layer="91"/>
+<junction x="101.6" y="81.28"/>
+</segment>
+</net>
+<net name="SCL" class="0">
+<segment>
+<pinref part="R1" gate="G$1" pin="1"/>
+<pinref part="C1" gate="G$1" pin="1"/>
+<wire x1="96.52" y1="101.6" x2="96.52" y2="91.44" width="0.1524" layer="91"/>
+<pinref part="U1" gate="A" pin="SCL"/>
+<wire x1="139.7" y1="101.6" x2="96.52" y2="101.6" width="0.1524" layer="91"/>
+<junction x="96.52" y="101.6"/>
+<wire x1="96.52" y1="101.6" x2="76.2" y2="101.6" width="0.1524" layer="91"/>
+<pinref part="X1" gate="-3" pin="S@1"/>
+<label x="81.28" y="101.6" size="1.778" layer="95"/>
+</segment>
+</net>
+<net name="SDA" class="0">
+<segment>
+<pinref part="R2" gate="G$1" pin="1"/>
+<pinref part="C2" gate="G$1" pin="1"/>
+<wire x1="109.22" y1="101.6" x2="109.22" y2="99.06" width="0.1524" layer="91"/>
+<pinref part="U1" gate="A" pin="SDA"/>
+<wire x1="109.22" y1="99.06" x2="109.22" y2="91.44" width="0.1524" layer="91"/>
+<wire x1="175.26" y1="104.14" x2="180.34" y2="104.14" width="0.1524" layer="91"/>
+<wire x1="180.34" y1="104.14" x2="180.34" y2="116.84" width="0.1524" layer="91"/>
+<wire x1="180.34" y1="116.84" x2="116.84" y2="116.84" width="0.1524" layer="91"/>
+<wire x1="116.84" y1="116.84" x2="116.84" y2="99.06" width="0.1524" layer="91"/>
+<wire x1="116.84" y1="99.06" x2="109.22" y2="99.06" width="0.1524" layer="91"/>
+<junction x="109.22" y="99.06"/>
+<wire x1="109.22" y1="99.06" x2="76.2" y2="99.06" width="0.1524" layer="91"/>
+<pinref part="X1" gate="-2" pin="S@1"/>
+<label x="81.28" y="99.06" size="1.778" layer="95"/>
+</segment>
+</net>
+<net name="N$3" class="0">
+<segment>
+<pinref part="R3" gate="G$1" pin="1"/>
+<pinref part="U1" gate="A" pin="A0"/>
+<wire x1="129.54" y1="101.6" x2="129.54" y2="96.52" width="0.1524" layer="91"/>
+<wire x1="129.54" y1="96.52" x2="139.7" y2="96.52" width="0.1524" layer="91"/>
+</segment>
+</net>
 </nets>
 </sheet>
