File: AquisitionExpansionModule/PCB/AcquisitionExpansionModule/AcquisitionExpansionModule.sch (EAGLE design)
At the start: 6 parts, among them U1 ADS1015IDGST, X1 87438-04

Commit message: designing PCB
designing PCB, edit schematic
Parts:
- removed SV1: (no value), con-lstb:MA04-1
- added X2: 87438-05, con-molex:87438-05
Connections:
- net GND: now also X2-1.S
- net N$1: now also X1-1.S; no longer X1-2.S
- net N$2: now also X1-2.S; no longer X1-3.S
- net N$3: now also X2-5.S; no longer SV1.1
- net N$4: now also X2-4.S; no longer SV1.2
- net N$5: now also X2-3.S; no longer SV1.3
- net N$6: now also X2-2.S; no longer SV1.4
- net VCC: now also X1-3.S; no longer X1-1.S
Other:
- moved on the sheet: X1-1, X1-2, X1-3, X1-4
Changed lines of the file:
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@@
 <?xml version="1.0" encoding="utf-8"?>
 <!DOCTYPE eagle SYSTEM "eagle.dtd">
-<eagle version="6.1">
+<eagle version="6.6.0">
 <drawing>
 <settings>
@@
 <part name="R1" library="resistor" deviceset="R-EU_" device="MELF0102W" value="10K"/>
 <part name="R2" library="resistor" deviceset="R-EU_" device="MELF0102W" value="10K"/>
-<part name="SV1" library="con-lstb" deviceset="MA04-1" device=""/>
 <part name="R3" library="resistor" deviceset="R-EU_" device="MELF0102W" value="10K"/>
 <part name="X1" library="con-molex" deviceset="87438-04" device=""/>
+<part name="X2" library="con-molex" deviceset="87438-05" device=""/>
+<part name="GND3" library="supply1" deviceset="GND" device=""/>
 </parts>
 <sheets>
@@
 <instance part="P+1" gate="VCC" x="101.6" y="124.46"/>
 <instance part="GND1" gate="1" x="101.6" y="86.36"/>
-<instance part="GND2" gate="1" x="170.18" y="106.68"/>
+<instance part="GND2" gate="1" x="170.18" y="104.14"/>
 <instance part="P+2" gate="VCC" x="167.64" y="137.16"/>
 <instance part="R1" gate="G$1" x="154.94" y="124.46" rot="R90"/>
 <instance part="R2" gate="G$1" x="162.56" y="124.46" rot="R90"/>
-<instance part="SV1" gate="1" x="81.28" y="101.6"/>
 <instance part="R3" gate="G$1" x="147.32" y="124.46" rot="R90"/>
-<instance part="X1" gate="-1" x="175.26" y="119.38"/>
-<instance part="X1" gate="-2" x="175.26" y="116.84"/>
-<instance part="X1" gate="-3" x="175.26" y="114.3"/>
-<instance part="X1" gate="-4" x="175.26" y="111.76"/>
+<instance part="X1" gate="-1" x="175.26" y="116.84"/>
+<instance part="X1" gate="-2" x="175.26" y="114.3"/>
+<instance part="X1" gate="-3" x="175.26" y="111.76"/>
+<instance part="X1" gate="-4" x="175.26" y="109.22"/>
+<instance part="X2" gate="-1" x="78.74" y="106.68" rot="MR0"/>
+<instance part="X2" gate="-2" x="78.74" y="104.14" rot="MR0"/>
+<instance part="X2" gate="-3" x="78.74" y="101.6" rot="MR0"/>
+<instance part="X2" gate="-4" x="78.74" y="99.06" rot="MR0"/>
+<instance part="X2" gate="-5" x="78.74" y="96.52" rot="MR0"/>
+<instance part="GND3" gate="1" x="83.82" y="91.44"/>
 </instances>
 <busses>
@@
 <segment>
 <pinref part="P+2" gate="VCC" pin="VCC"/>
-<wire x1="172.72" y1="119.38" x2="167.64" y2="119.38" width="0.1524" layer="91"/>
-<wire x1="167.64" y1="119.38" x2="167.64" y2="129.54" width="0.1524" layer="91"/>
+<wire x1="167.64" y1="111.76" x2="167.64" y2="129.54" width="0.1524" layer="91"/>
 <pinref part="R2" gate="G$1" pin="2"/>
 <wire x1="167.64" y1="129.54" x2="167.64" y2="134.62" width="0.1524" layer="91"/>
@@
 <wire x1="147.32" y1="129.54" x2="154.94" y2="129.54" width="0.1524" layer="91"/>
 <junction x="154.94" y="129.54"/>
-<pinref part="X1" gate="-1" pin="S"/>
+<pinref part="X1" gate="-3" pin="S"/>
+<wire x1="167.64" y1="111.76" x2="172.72" y2="111.76" width="0.1524" layer="91"/>
 </segment>
 </net>
@@
 <segment>
 <pinref part="GND2" gate="1" pin="GND"/>
-<wire x1="172.72" y1="111.76" x2="170.18" y2="111.76" width="0.1524" layer="91"/>
-<wire x1="170.18" y1="111.76" x2="170.18" y2="109.22" width="0.1524" layer="91"/>
+<wire x1="172.72" y1="109.22" x2="170.18" y2="109.22" width="0.1524" layer="91"/>
+<wire x1="170.18" y1="109.22" x2="170.18" y2="106.68" width="0.1524" layer="91"/>
 <pinref part="X1" gate="-4" pin="S"/>
+</segment>
+<segment>
+<pinref part="X2" gate="-1" pin="S"/>
+<pinref part="GND3" gate="1" pin="GND"/>
+<wire x1="81.28" y1="106.68" x2="83.82" y2="106.68" width="0.1524" layer="91"/>
+<wire x1="83.82" y1="106.68" x2="83.82" y2="93.98" width="0.1524" layer="91"/>
 </segment>
 </net>
@@
 <wire x1="144.78" y1="116.84" x2="162.56" y2="116.84" width="0.1524" layer="91"/>
 <pinref part="R2" gate="G$1" pin="1"/>
-<wire x1="162.56" y1="116.84" x2="172.72" y2="116.84" width="0.1524" layer="91"/>
 <wire x1="162.56" y1="119.38" x2="162.56" y2="116.84" width="0.1524" layer="91"/>
+<pinref part="X1" gate="-1" pin="S"/>
+<wire x1="172.72" y1="116.84" x2="162.56" y2="116.84" width="0.1524" layer="91"/>
 <junction x="162.56" y="116.84"/>
-<pinref part="X1" gate="-2" pin="S"/>
 </segment>
 </net>
 <net name="N$2" class="0">
 <segment>
-<wire x1="172.72" y1="114.3" x2="154.94" y2="114.3" width="0.1524" layer="91"/>
+<wire x1="154.94" y1="119.38" x2="154.94" y2="114.3" width="0.1524" layer="91"/>
 <wire x1="154.94" y1="114.3" x2="154.94" y2="78.74" width="0.1524" layer="91"/>
 <wire x1="154.94" y1="78.74" x2="93.98" y2="78.74" width="0.1524" layer="91"/>
@@
 <wire x1="93.98" y1="109.22" x2="104.14" y2="109.22" width="0.1524" layer="91"/>
 <pinref part="R1" gate="G$1" pin="1"/>
-<wire x1="154.94" y1="119.38" x2="154.94" y2="114.3" width="0.1524" layer="91"/>
+<pinref part="X1" gate="-2" pin="S"/>
+<wire x1="172.72" y1="114.3" x2="154.94" y2="114.3" width="0.1524" layer="91"/>
 <junction x="154.94" y="114.3"/>
-<pinref part="X1" gate="-3" pin="S"/>
 </segment>
 </net>
 <net name="N$3" class="0">
 <segment>
-<pinref part="SV1" gate="1" pin="1"/>
 <pinref part="U1" gate="A" pin="NC"/>
 <wire x1="104.14" y1="93.98" x2="101.6" y2="93.98" width="0.1524" layer="91"/>
 <wire x1="101.6" y1="93.98" x2="101.6" y2="96.52" width="0.1524" layer="91"/>
-<wire x1="101.6" y1="96.52" x2="88.9" y2="96.52" width="0.1524" layer="91"/>
+<wire x1="101.6" y1="96.52" x2="81.28" y2="96.52" width="0.1524" layer="91"/>
+<pinref part="X2" gate="-5" pin="S"/>
 </segment>
 </net>
 <net name="N$4" class="0">
 <segment>
-<pinref part="SV1" gate="1" pin="2"/>
 <pinref part="U1" gate="A" pin="NC_2"/>
 <wire x1="104.14" y1="96.52" x2="104.14" y2="99.06" width="0.1524" layer="91"/>
-<wire x1="104.14" y1="99.06" x2="88.9" y2="99.06" width="0.1524" layer="91"/>
+<wire x1="104.14" y1="99.06" x2="81.28" y2="99.06" width="0.1524" layer="91"/>
+<pinref part="X2" gate="-4" pin="S"/>
 </segment>
 </net>
 <net name="N$5" class="0">
 <segment>
-<pinref part="SV1" gate="1" pin="3"/>
 <pinref part="U1" gate="A" pin="AIN1"/>
-<wire x1="104.14" y1="101.6" x2="88.9" y2="101.6" width="0.1524" layer="91"/>
+<wire x1="104.14" y1="101.6" x2="81.28" y2="101.6" width="0.1524" layer="91"/>
+<pinref part="X2" gate="-3" pin="S"/>
 </segment>
 </net>
 <net name="N$6" class="0">
 <segment>
-<pinref part="SV1" gate="1" pin="4"/>
 <pinref part="U1" gate="A" pin="AIN0"/>
-<wire x1="104.14" y1="104.14" x2="88.9" y2="104.14" width="0.1524" layer="91"/>
-</segment>
-</net>
+<wire x1="104.14" y1="104.14" x2="81.28" y2="104.14" width="0.1524" layer="91"/>
+<pinref part="X2" gate="-2" pin="S"/>
+</segment>
+</net>
